File: KiCad/Systems&Electronics.kicad_sch (KiCad schematic)
At the start: 39 parts, among them U13 AD8495, U14 AD8495, U15 AD8495, U16 AD8495, U3 MAX485E, U4 MAX485E

Commit message: Firmware Refactor (Untested)
Parts:
- renumbered Solenoid3 to Fuel, Solenoid2 to FuelPressure, Solenoid1 to NitrogenFlush, Solenoid4 to Oxidizer
Connections:
- net at Oxidizer. (-): now also 5V Relay4. (NO), D2.2 (A), D3.1 (K), Fuel. (-), FuelPressure. (-), NitrogenFlush. (-); no longer 5V Relay5. (NO)
- net at Pressure_Transducer1. (VCC), Pressure_Transducer2. (VCC), Pressure_Transducer3. (VCC)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: now also A1.GND1 (GND); no longer A1.5V3 (5V)
- new net: 5V Relay1. (NO), 5V Relay2. (NO), 5V Relay3. (NO), 5V Relay4. (NO), 5V Relay5. (NO), A1.GND5 (GND), D4.1 (K), D5.1 (K), D6.1 (K)
- new net: 5V Relay1. (NO), 5V Relay2. (NO), 5V Relay3. (NO), 5V Relay5. (NO), A1.5V4 (5V)
- new net: 5V Relay5. (NO), Oxidizer. (-)
- new net: 5V Relay1. (NO), NitrogenFlush. (-)
- new net: A1.5V3 (5V), Pressure_Transducer1. (VCC), Pressure_Transducer2. (VCC), Pressure_Transducer3. (VCC), Pressure_Transducer4. (VCC), Pressure_Transducer5. (VCC), Pressure_Transducer6. (VCC)
- new net: HX711_Board1. (VCC), Load_Cell1. (VCC) (x3)
Changed lines of the file:
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@@
 	)
 	(symbol
+		(lib_name "Solenoids:Solenoid")
 		(lib_id "Solenoids:Solenoid")
 		(at 273.05 128.27 0)
@@
 		(dnp no)
 		(fields_autoplaced yes)
-		(property "Reference" "Solenoid4"
+		(property "Reference" "Oxidizer"
 			(at 273.05 120.65 0)
 			(effects
@@
 			(project "Systems&Electronics"
 				(path "/4e05caf8-77e4-4a22-9a05-51fcca8e50ff"
-					(reference "Solenoid4")
+					(reference "Oxidizer")
 					(unit 1)
 				)
@@
 	)
 	(symbol
+		(lib_name "Solenoids:Solenoid")
 		(lib_id "Solenoids:Solenoid")
 		(at 251.46 128.27 0)
@@
 		(dnp no)
 		(fields_autoplaced yes)
-		(property "Reference" "Solenoid3"
+		(property "Reference" "Fuel"
 			(at 251.46 120.65 0)
 			(effects
@@
 			(project ""
 				(path "/4e05caf8-77e4-4a22-9a05-51fcca8e50ff"
-					(reference "Solenoid3")
+					(reference "Fuel")
 					(unit 1)
 				)
@@
 	)
 	(symbol
+		(lib_name "Solenoids:Solenoid")
 		(lib_id "Solenoids:Solenoid")
 		(at 195.58 128.27 0)
@@
 		(dnp no)
 		(fields_autoplaced yes)
-		(property "Reference" "Solenoid1"
+		(property "Reference" "NitrogenFlush"
 			(at 195.58 120.65 0)
 			(effects
@@
 			(project ""
 				(path "/4e05caf8-77e4-4a22-9a05-51fcca8e50ff"
-					(reference "Solenoid1")
+					(reference "NitrogenFlush")
 					(unit 1)
 				)
@@
 	)
 	(symbol
+		(lib_name "Solenoids:Solenoid")
 		(lib_id "Solenoids:Solenoid")
 		(at 223.52 128.27 0)
@@
 		(dnp no)
 		(fields_autoplaced yes)
-		(property "Reference" "Solenoid2"
+		(property "Reference" "FuelPressure"
 			(at 223.52 120.65 0)
 			(effects
@@
 			(project ""
 				(path "/4e05caf8-77e4-4a22-9a05-51fcca8e50ff"
-					(reference "Solenoid2")
-					(unit 1)
-				)
+					(reference "FuelPressure")
+					(unit 1)
+				)
