File: KiCad/Engine_Mainboard/Control_Room.kicad_sch (KiCad schematic)
At the start: 4 parts, among them U1 MAX485E, U2 MAX485E

Commit message: Finishing touches, added redundant power terminals, and reset button.
Parts:
- removed J_USB_DATA1: TX_RX, symbol Connector:Screw_Terminal_01x02
- removed J_USB_POWER1: Power, symbol Connector:Screw_Terminal_01x02
- removed U1, U2: MAX485E, symbol Interface_UART:MAX485E
Other:
- note removed: "1.1.0"
- note removed: "RPI Spaceflight Society"
- note removed: "RPU V1 Test Stand Electronics"
- note removed: "September 10, 2024"
